File: parts/dmx-controller/pcb/dmx-controller.kicad_pcb (KiCad board)
At the start: 2 copper layers, 98 x 50 mm, 17 parts, among them J2 PWR IN, SW2 SW_SPDT, U1 ESP32 Wemos D1 Mini

Commit message: new version of KiCad
Routing:
- net GND: track 0.00 -> 159.1 mm
- net /3V3: track 0.00 -> 89.9 mm
- net Net-(ETH2-RST): track 0.00 -> 55.2 mm, vias 0 -> 1
- net Net-(RS485_MODULE_J3-RXD): track 0.00 -> 49.1 mm, vias 0 -> 1
- net Net-(RS485_MODULE_J3-TXD): track 0.00 -> 45.5 mm, vias 0 -> 1
- net Net-(12V_BUCK1-+12Vin): track 0.00 -> 35.0 mm, vias 0 -> 1
- net Net-(RS485_MODULE_J1-RXD): track 0.00 -> 33.5 mm
- net Net-(RS485_MODULE_J1-TXD): track 0.00 -> 29.9 mm
- net SHIELD: track 0.00 -> 25.4 mm
- net /5V: track 0.00 -> 25.2 mm
- net Net-(ETH2-MISO): track 0.00 -> 23.5 mm
- net /SCK: track 0.00 -> 20.8 mm, vias 0 -> 1
- net /MOSI: track 0.00 -> 19.9 mm
- net /INT: track 0.00 -> 18.7 mm, vias 0 -> 1
- net /CS: track 0.00 -> 14.4 mm
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