File: parts/poe-injector/pcb/poe-injector.kicad_sch (KiCad schematic)
At the start: 12 parts, among them SW2 SW_SPDT

Commit message: pcb revisions to update to better RJ45 jack, update QR code.
Parts:
- 1GB_ETH_IN1, 1GB_POE_ETH_OUT1: footprint Connector_RJ:RJ45_Ninigi_GE -> Connector_RJ:RJ45_Amphenol_RJHSE5380
