File: parts/env-sensor/pcb/mcu/env-sensor-mcu.kicad_pcb (KiCad board)
At the start: 2 copper layers, 53.3 x 33 mm, 9 parts, among them J1 Conn_02x08_Top_Bottom, J2 Conn_02x08_Top_Bottom, J3 Conn_01x01_Shielded

Commit message: refresh env-sensor as I screwed up the pinouts in the last fab run.
Other:
- board text added: "(C) 2026 ARKADIA HOUSE Env Sensor MCU rev 1.4"
- board text added: "ILL 3V3 SDA GND SCL"
- board text removed: "(C) 2026 ARKADIA HOUSE Env Sensor MCU rev 1.3"
- board text removed: "SCL GND SDA 3V3 ILL"

Commit message: rev QR code
Other:
- board text added: "(C) 2026 ARKADIA HOUSE Env Sensor MCU rev 1.4.1"
- board text removed: "(C) 2026 ARKADIA HOUSE Env Sensor MCU rev 1.4"
