File: parts/keypad/pcb/keypad.kicad_pcb (KiCad board)
At the start: 2 copper layers, 95 x 74.5 mm, 22 parts, among them J1 Conn_02x10_Top_Bottom, J2 1x10, J3 To MCU, J4 To DISP, SW1 SW_Push, SW10 SW_Push, SW2 SW_Push, SW3 SW_Push, SW4 SW_Push, SW5 SW_Push, SW6 SW_Push, SW7 SW_Push, SW8 SW_Push, SW9 SW_Push

Commit message: revise QR code
Other:
- board text added: "(C) 2026 ARKADIA HOUSE Keypad Display rev 01.5.1"
- board text removed: "(C) 2026 ARKADIA HOUSE Keypad Display rev 01.5"

Commit message: update 1.5.2 waiting to build another before fabbing this rev.
Routing:
- net /COM: track 299.8 -> 297.7 mm
- net /N$10: track 25.0 -> 24.4 mm
Other:
- board text added: "(C) 2026 ARKADIA HOUSE Keypad Display rev 01.5.2"
- board text removed: "(C) 2026 ARKADIA HOUSE Keypad Display rev 01.5.1"
