File: parts/keypad/pcb/keypad.kicad_sch (KiCad schematic)
At the start: 14 parts, among them J1 Conn_02x10_Top_Bottom, J2 1x10, J3 To SENSOR HUB, J4 To DISPLAY MODULE, SW1 SW_Push, SW10 SW_Push, SW2 SW_Push, SW3 SW_Push, SW4 SW_Push, SW5 SW_Push, SW6 SW_Push, SW7 SW_Push, SW8 SW_Push, SW9 SW_Push

Commit message: update connector to hub to match hub pinouts
Parts:
- removed J3: To SENSOR HUB, Connector_PinHeader_2.54mm:PinHeader_1x04_P2.54mm_Horizontal, symbol Connector_Generic:Conn_01x04
- added TO_HUB1: Conn_01x05, Connector_PinHeader_2.54mm:PinHeader_1x05_P2.54mm_Horizontal, symbol Connector_Generic:Conn_01x05
Connections:
- net GND: now also TO_HUB1.3 (Pin_3)
- net at J2.8 (SCL), J4.3 (SCL): now also TO_HUB1.1 (Pin_1)
- net at J2.7 (SDA), J4.4 (SDA): now also TO_HUB1.2 (Pin_2)
- net at J2.10 (3V3), J4.2 (3V3): now also TO_HUB1.5 (Pin_5)
- no-connect marks 0 -> 1
Changed lines of the file:
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@@
+	)
+	(junction
+		(at 171.45 113.03)
+		(diameter 0)
+		(color 0 0 0 0)
 	)
 	(junction
@@
 	)
 	(junction
-		(at 171.45 113.03)
-		(diameter 0)
-		(color 0 0 0 0)
-	)
-	(junction
 		(at 25.4 67.31)
 		(diameter 0)
@@
 	)
 	(junction
-		(at 176.53 110.49)
-		(diameter 0)
-		(color 0 0 0 0)
-	)
-	(junction
 		(at 25.4 41.91)
 		(diameter 0)
@@
 	)
 	(junction
+		(at 181.61 110.49)
+		(diameter 0)
+		(color 0 0 0 0)
+	)
+	(junction
 		(at 173.99 115.57)
 		(diameter 0)
@@
 		(color 0 0 0 0)
 	)
+	(no_connect
+		(at 179.07 154.94)
+	)
+	(wire
+		(pts
+			(xy 176.53 147.32) (xy 179.07 147.32)
+		)
+		(stroke
+			(width 0)
+			(type default)
+		)
+	)
 	(wire
 		(pts
@@
 	(wire
 		(pts
-			(xy 176.53 101.6) (xy 176.53 110.49)
-		)
-		(stroke
-			(width 0)
-			(type default)
-		)
-	)
-	(wire
-		(pts
 			(xy 25.4 93.98) (xy 77.47 93.98)
 		)
@@
 	(wire
 		(pts
-			(xy 176.53 101.6) (xy 181.61 101.6)
-		)
-		(stroke
-			(width 0)
-			(type default)
-		)
-	)
-	(wire
-		(pts
 			(xy 25.4 91.44) (xy 25.4 93.98)
 		)
@@
 	(wire
 		(pts
+			(xy 179.07 107.95) (xy 179.07 147.32)
+		)
+		(stroke
+			(width 0)
+			(type default)
+		)
+	)
+	(wire
+		(pts
 			(xy 176.53 15.24) (xy 176.53 55.88)
 		)
@@
 	(wire
 		(pts
+			(xy 176.53 147.32) (xy 176.53 154.94)
+		)
+		(stroke
+			(width 0)
+			(type default)
+		)
+	)
+	(wire
+		(pts
 			(xy 179.07 95.25) (xy 179.07 92.71)
 		)
@@
 	(wire
 		(pts
+			(xy 173.99 115.57) (xy 173.99 154.94)
+		)
+		(stroke
+			(width 0)
+			(type default)
+		)
+	)
+	(wire
+		(pts
 			(xy 171.45 20.32) (xy 171.45 55.88)
 		)
@@
 	(wire
 		(pts
-			(xy 171.45 113.03) (xy 171.45 124.46)
-		)
-		(stroke
-			(width 0)
-			(type default)
-		)
-	)
-	(wire
-		(pts
 			(xy 148.59 34.29) (xy 148.59 22.86)
 		)
@@
 	(wire
 		(pts
-			(xy 179.07 107.95) (xy 179.07 124.46)
-		)
-		(stroke
-			(width 0)
-			(type default)
-		)
-	)
-	(wire
-		(pts
 			(xy 77.47 64.77) (xy 77.47 67.31)
 		)
@@
 	(wire
 		(pts
-			(xy 173.99 115.57) (xy 173.99 124.46)
+			(xy 181.61 110.49) (xy 203.2 110.49)
 		)
 		(stroke
@@
 	(wire
 		(pts
-			(xy 181.61 92.71) (xy 181.61 101.6)
+			(xy 181.61 92.71) (xy 181.61 110.49)
 		)
 		(stroke
@@
 	(wire
 		(pts
+			(xy 181.61 110.49) (xy 181.61 154.94)
+		)
+		(stroke
+			(width 0)
+			(type default)
+		)
+	)
+	(wire
+		(pts
 			(xy 138.43 34.29) (xy 138.43 41.91)
 		)
@@
 	(wire
 		(pts
-			(xy 176.53 110.49) (xy 176.53 124.46)
-		)
-		(stroke
-			(width 0)
-			(type default)
-		)
-	)
-	(wire
-		(pts
 			(xy 55.88 73.66) (xy 154.94 73.66)
 		)
@@
 	(wire
 		(pts
-			(xy 176.53 110.49) (xy 203.2 110.49)
-		)
-		(stroke
-			(width 0)
-			(type default)
-		)
-	)
-	(wire
-		(pts
 			(xy 171.45 113.03) (xy 203.2 113.03)
 		)
@@
 	(wire
 		(pts
+			(xy 87.63 77.47) (xy 176.53 77.47)
+		)
+		(stroke
+			(width 0)
+			(type default)
+		)
+	)
+	(wire
+		(pts
 			(xy 171.45 97.79) (xy 171.45 113.03)
 		)
@@
 	(wire
 		(pts
-			(xy 87.63 77.47) (xy 176.53 77.47)
-		)
-		(stroke
-			(width 0)
-			(type default)
-		)
-	)
-	(wire
-		(pts
 			(xy 106.68 91.44) (xy 106.68 96.52)
 		)
@@
 		(pts
 			(xy 87.63 34.29) (xy 87.63 17.78)
+		)
+		(stroke
+			(width 0)
+			(type default)
+		)
+	)
+	(wire
+		(pts
+			(xy 171.45 113.03) (xy 171.45 154.94)
 		)
 		(stroke
@@
 		)
 	)
+	(label "SDA"
+		(at 175.26 161.29 270)
+		(effects
+			(font
+				(size 1.27 1.27)
+			)
+			(justify right bottom)
+		)
+	)
 	(label "N$3"
 		(at 116.84 34.29 0)
@@
 		)
 	)
+	(label "5V"
+		(at 180.34 161.29 270)
+		(effects
+			(font
+				(size 1.27 1.27)
+			)
+			(justify right bottom)
+		)
+	)
 	(label "N$9"
 		(at 87.63 91.44 0)
@@
 		)
 	)
+	(label "SCL"
+		(at 172.72 161.29 270)
+		(effects
+			(font
+				(size 1.27 1.27)
+			)
+			(justify right bottom)
+		)
+	)
 	(label "N$6"
 		(at 87.63 64.77 0)
@@
 			)
 			(justify right bottom)
-		)
-	)
-	(symbol
-		(lib_id "Connector_Generic:Conn_01x04")
-		(at 173.99 129.54 90)
-		(mirror x)
-		(unit 1)
-		(body_style 1)
-		(exclude_from_sim no)
-		(in_bom yes)
-		(on_board yes)
-		(in_pos_files yes)
-		(dnp no)
-		(property "Reference" "J3"
-			(at 182.626 128.524 0)
-			(show_name no)
-			(do_not_autoplace no)
-			(effects
-				(font
-					(size 1.27 1.27)
-				)
-				(justify left)
-			)
-		)
-		(property "Value" "To SENSOR HUB"
-			(at 182.88 137.414 90)
-			(show_name no)
-			(do_not_autoplace no)
-			(effects
-				(font
-					(size 1.27 1.27)
-				)
-				(justify left)
-			)
-		)
-		(property "Footprint" "Connector_PinHeader_2.54mm:PinHeader_1x04_P2.54mm_Horizontal"
-			(at 173.99 129.54 0)
-			(hide yes)
-			(show_name no)
-			(do_not_autoplace no)
-			(effects
-				(font
-					(size 1.27 1.27)
-				)
-			)
-		)
-		(property "Datasheet" ""
-			(at 173.99 129.54 0)
-			(hide yes)
-			(show_name no)
-			(do_not_autoplace no)
-			(effects
-				(font
-					(size 1.27 1.27)
-				)
-			)
-		)
-		(property "Description" "Generic connector, single row, 01x04, script generated (kicad-library-utils/schlib/autogen/connector/)"
-			(at 173.99 129.54 0)
-			(hide yes)
-			(show_name no)
-			(do_not_autoplace no)
-			(effects
-				(font
-					(size 1.27 1.27)
-				)
-			)
-		)
-		(pin "4"
-		)
-		(pin "1"
-		)
-		(pin "3"
-		)
-		(pin "2"
-		)
-		(instances
-			(project "keypad"
-				(path "/8a716d07-f2fb-4734-9a1b-56d3b5fc3e34"
-					(reference "J3")
-					(unit 1)
-				)
-			)
 		)
 	)
@@
 					(unit 1)
 				)
+			)
+		)
+	)
+	(symbol
+		(lib_id "Connector_Generic:Conn_01x05")
+		(at 176.53 160.02 90)
+		(mirror x)
+		(unit 1)
+		(body_style 1)
+		(exclude_from_sim no)
+		(in_bom yes)
+		(on_board yes)
+		(in_pos_files yes)
+		(dnp no)
+		(property "Reference" "TO_HUB1"
+			(at 185.166 153.162 0)
+			(show_name no)
+			(do_not_autoplace no)
+			(effects
+				(font
+					(size 1.27 1.27)
+				)
+				(justify left)
+			)
+		)
+		(property "Value" "Conn_01x05"
+			(at 177.7999 162.56 0)
+			(hide yes)
+			(show_name no)
+			(do_not_autoplace no)
+			(effects
+				(font
+					(size 1.27 1.27)
+				)
+				(justify left)
+			)
+		)
+		(property "Footprint" "Connector_PinHeader_2.54mm:PinHeader_1x05_P2.54mm_Horizontal"
+			(at 176.53 160.02 0)
+			(hide yes)
+			(show_name no)
+			(do_not_autoplace no)
+			(effects
+				(font
+					(size 1.27 1.27)
+				)
+			)
+		)
+		(property "Datasheet" ""
+			(at 176.53 160.02 0)
+			(hide yes)
+			(show_name no)
+			(do_not_autoplace no)
+			(effects
+				(font
+					(size 1.27 1.27)
+				)
+			)
+		)
+		(property "Description" "Generic connector, single row, 01x05, script generated (kicad-library-utils/schlib/autogen/connector/)"
+			(at 176.53 160.02 0)
+			(hide yes)
+			(show_name no)
+			(do_not_autoplace no)
+			(effects
+				(font
+					(size 1.27 1.27)
+				)
+			)
+		)
+		(pin "1"
+		)
+		(pin "2"
+		)
+		(pin "4"
+		)
+		(pin "3"
+		)
+		(pin "5"
+		)
+		(instances
+			(project "keypad"
+				(path "/8a716d07-f2fb-4734-9a1b-56d3b5fc3e34"
+					(reference "TO_HUB1")
+					(unit 1)
+				)
