File: parts/sensor-hub/hub/pcb/sensor-hub.kicad_pcb (KiCad board)
At the start: 2 copper layers, 85.7 x 47 mm, 13 parts, among them J1 MPT1584 buck, J2 PWR IN, SW2 SW_SPDT, U1 ESP32 Wemos D1 Mini

Commit message: update QR code
Other:
- board text added: "Sensor Hub rev 6.9.1"
- board text removed: "Sensor Hub rev 6.9"

Commit message: sensor hub rev 6.9.2
Routing:
- net GND: track 211.0 -> 208.5 mm
- net Net-(ETH2-RST): track 81.3 -> 80.0 mm
- net /DL1_SENSE: track 32.1 -> 30.9 mm
- net /DS1_SENSE: track 25.5 -> 24.4 mm
- net /5V: track 111.5 -> 110.9 mm
- net /SCK: track 58.6 -> 58.0 mm
- net /INT: track 59.9 -> 59.3 mm
Other:
- board text added: "Sensor Hub rev 6.9.2"
- board text removed: "Sensor Hub rev 6.9.1"
