File: parts/strip-led-controller/pcb/strip-led-controller.kicad_sch (KiCad schematic)
At the start: 11 parts, among them J1 BUCK_IN, J2 PWR IN, J3 BUCK_OUT, SW2 SW_SPDT, U1 ESP32 Wemos D1 Mini

Commit message: change strip connectors to screw terminals
Parts:
- L1, L2: footprint Connector_PinHeader_2.54mm:PinHeader_1x04_P2.54mm_Horizontal -> TerminalBlock:TerminalBlock_Xinya_XY308-2.54-4P_1x04_P2.54mm_Horizontal
